File: KiCad/pelletpirate_V5/PelletPirate_V5.kicad_sch (KiCad schematic)
At the start: 141 parts, among them J1 SJ1-3523NG_Jack_PP, J2 SJ1-3523NG_Jack_PP, J3 SJ1-3523NG_Jack_PP, J4 SJ1-3523NG_Jack_PP, J5 SJ1-3523NG_Jack_PP, J6 Conn_01x04, J7 Conn_01x04_Socket, J8 USB4105-GF-A_fly, J9 Conn_01x02, T1 BTA12-Triac, T2 BTA12-Triac, T3 BTA12-Triac, T4 BTA12-600BWRG, U1 USBLC6-2SC6, U3 H11AA1M

Commit message: V5 Phase A complete: S3 schematic surgery, ERC clean
DevKit rails (ESP_J2/ESP_J3) deleted; F1 onboard fuse RETAINED (in
series with proven AC copper; inline panel fuse is supplementary).
S3/USB/ZC/hopper blocks stitched to V2 nets by label — SDO line
standardized to ALL_SDO fleet-wide (was MAX_SDO on V2). Fan channel
converted by-the-book: true MOC3053M symbol (full MPN/DigiKey fields)
wired in and re-referenced as MOC3 so Update-PCB maps onto the
existing AC-island footprint; R9 330->180 ohm with real part fields
(anti-sulfur pulse-withstanding 0805 per V4 BOM). NC flags verified
on IO35/36/37 (PSRAM) and unused pads. ERC: 0.

Co-Authored-By: Claude Fable 5 <noreply@anthropic.com>
Parts:
- removed ESP_J2: PelletPirate_J2_01toJ2_19, ESP32-Footprint-PelletPirate-02x19x2=39:PinHeader_J2x19_P2.54mm_Vertical_PelletPirate, symbol ESP32-DEVKITC-32E_PelletPirate:PelletPirate_J2_01toJ2_19_Socket
- removed ESP_J3: PelletPirate_J3_01toJ3_19, ESP32-Footprint-PelletPirate-02x19x2=39:PinHeader_J3x19_P2.54mm_Vertical_PelletPirate, symbol ESP32-DEVKITC-32E_PelletPirate:PelletPirate_J3_01toJ3_19_Socket
- removed MOC3: MOC3063M, MOC3063M-PP2:MOC3063M-PP2, symbol MOC3063M-PP2:MOC3063M-PelletPirate
- removed R13, R14, R18, R29, R30, R31: 10KΩ, Resistor_SMD:R_0805_2012Metric_Pad1.20x1.40mm_HandSolder, symbol Device:R_US
- removed R28, R6: 360Ω 1/4W, Resistor_SMD:R_1206_3216Metric, symbol Device:R_US
- removed R9: 330Ω, Resistor_SMD:R_0805_2012Metric_Pad1.20x1.40mm_HandSolder, symbol Device:R_US
- removed T3: BTA12-Triac, Package_TO_SOT_THT:TO-220-3_Vertical, symbol BTA12-600BWRG:BTA12-600BW-PelletPirate
- removed WirePad5: FAN(L), Connector_Wire:SolderWire-2.5sqmm_1x01_D2.4mm_OD3.6mm, symbol Connector:Conn_01x01_Pin
- renumbered MOC4 to MOC3, R46 to R28, R11 to R6, R10 to R9, T4 to T3
Connections:
- net MAX_SDO is gone; now on net ALL_SDO: FPC1.30, MAX1.14 (SDO), MAX2.14 (SDO), MAX3.14 (SDO), MAX4.14 (SDO), MAX5.14 (SDO)
- net AC-LOAD: now also R6.1, T3.2 (A2)
- net at C3.2: now also R28.2, T3.1 (A1), WirePad6.1 (Pin_1)
- no-connect marks 37 -> 24
Other:
- moved on the sheet: C17, C21, C22, C23, C24, C25, C26, C27, C28, C29, C30, C31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

Commit message: V5 Phase B/C checkpoint: Update-PCB applied, placement in progress
Board now carries the full V5 netlist: S3/USB/ZC/hopper/switch/LED
footprints on board, SDO net renamed to ALL_SDO across existing copper
(tracks preserved), fan channel = MOC3053M with verified Panasonic
ERJ-UP6F1800V drive resistors, DNP flags cleared, WirePad5 relinked.
New parts rough-placed; nets locked next, then arrangement and routing.
FPC1 decision: moving to top-left (side B) pending flex-reach check.

Hard-won process lessons this session: Update-PCB must run with
re-link-by-reference CHECKED (UUID matching deletes re-associated
footprints); preview dialogs can serve stale reports — regenerate
fresh after schematic saves; editor memory can diverge from disk after
undo chains — verify against the file and close-without-save to recover.

Co-Authored-By: Claude Fable 5 <noreply@anthropic.com>
Parts:
- Earth1, WirePad1, WirePad2: footprint Connector_Wire:SolderWire-2.5sqmm_1x01_D2.4mm_OD4.4mm -> Connector_Wire:SolderWire-1.5sqmm_1x01_D1.7mm_OD3mm
- PS1: footprint PBO-5F-12_PP_Try2:PBO-5F-12_pp2 -> NewPBO-5F-12-try:CONV_PBO-5F-12_AUDIT_FLYMAN
- WirePad3, WirePad4: footprint Connector_Wire:SolderWire-2.5sqmm_1x01_D2.4mm_OD3.6mm -> Connector_Wire:SolderWire-1.5sqmm_1x01_D1.7mm_OD3mm
- renumbered R33 to R32, R34 to R33, R35 to R34, R38 to R35, R41 to R36, R42 to R37, R43 to R38, R45 to R41, R44 to R42, R47 to R43, R36 to R44, R32 to R45, R37 to R47, WirePad6 to WirePad5
Connections:
- net at C41.2, ESP1.22 (IO14): no longer R47.1
- net at J9.1 (Pin_1), R40.2: no longer R47.2
Other:
- moved on the sheet: R47
Changed lines of the file:
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@@
 		(in_pos_files yes)
 		(dnp no)
-		(property "Reference" "R47"
+		(property "Reference" "R43"
 			(at 86.106 307.594 0)
 			(show_name no)
@@
 			(project "PelletPirate_V5"
 				(path "/0182ac56-03c6-4c14-8ead-12e31828f094"
-					(reference "R47")
+					(reference "R43")
 					(unit 1)
 				)
@@
 		(in_pos_files yes)
 		(dnp no)
-		(property "Reference" "R41"
+		(property "Reference" "R36"
 			(at 254.254 213.868 0)
 			(show_name no)
@@
 			(project "PelletPirate_V5"
 				(path "/0182ac56-03c6-4c14-8ead-12e31828f094"
-					(reference "R41")
+					(reference "R36")
 					(unit 1)
 				)
@@
 		(in_pos_files yes)
 		(dnp no)
-		(property "Reference" "R33"
+		(property "Reference" "R32"
 			(at 168.402 201.676 0)
 			(show_name no)
@@
 			(project "PelletPirate_V5"
 				(path "/0182ac56-03c6-4c14-8ead-12e31828f094"
-					(reference "R33")
+					(reference "R32")
 					(unit 1)
 				)
@@
 		(in_pos_files yes)
 		(dnp no)
-		(property "Reference" "R43"
+		(property "Reference" "R38"
 			(at 303.784 202.438 0)
 			(show_name no)
@@
 			(project "PelletPirate_V5"
 				(path "/0182ac56-03c6-4c14-8ead-12e31828f094"
-					(reference "R43")
+					(reference "R38")
 					(unit 1)
 				)
@@
 			)
 		)
-		(property "Footprint" "Connector_Wire:SolderWire-2.5sqmm_1x01_D2.4mm_OD3.6mm"
+		(property "Footprint" "Connector_Wire:SolderWire-1.5sqmm_1x01_D1.7mm_OD3mm"
 			(at 99.06 158.75 0)
 			(hide yes)
@@
 		(in_pos_files yes)
 		(dnp no)
-		(property "Reference" "R45"
+		(property "Reference" "R41"
 			(at 41.402 304.8 90)
 			(show_name no)
@@
 			(project "PelletPirate_V5"
 				(path "/0182ac56-03c6-4c14-8ead-12e31828f094"
-					(reference "R45")
+					(reference "R41")
 					(unit 1)
 				)
@@
 		(in_pos_files yes)
 		(dnp no)
-		(property "Reference" "R42"
+		(property "Reference" "R37"
 			(at 285.496 202.438 0)
 			(show_name no)
@@
 			(project "PelletPirate_V5"
 				(path "/0182ac56-03c6-4c14-8ead-12e31828f094"
-					(reference "R42")
+					(reference "R37")
 					(unit 1)
 				)
@@
 			)
 		)
-		(property "Footprint" "Connector_Wire:SolderWire-2.5sqmm_1x01_D2.4mm_OD4.4mm"
+		(property "Footprint" "Connector_Wire:SolderWire-1.5sqmm_1x01_D1.7mm_OD3mm"
 			(at 63.5 46.99 0)
 			(hide yes)
@@
 			)
 		)
-		(property "Footprint" "Connector_Wire:SolderWire-2.5sqmm_1x01_D2.4mm_OD4.4mm"
+		(property "Footprint" "Connector_Wire:SolderWire-1.5sqmm_1x01_D1.7mm_OD3mm"
 			(at 62.23 58.42 0)
 			(hide yes)
@@
 		(in_pos_files yes)
 		(dnp no)
-		(property "Reference" "R35"
+		(property "Reference" "R34"
 			(at 179.578 201.422 0)
 			(show_name no)
@@
 			(project "PelletPirate_V5"
 				(path "/0182ac56-03c6-4c14-8ead-12e31828f094"
-					(reference "R35")
+					(reference "R34")
 					(unit 1)
 				)
@@
 	(symbol
 		(lib_id "Device:R_US")
-		(at 191.77 231.14 0)
-		(mirror y)
+		(at 191.77 231.14 270)
+		(mirror x)
 		(unit 1)
 		(body_style 1)
@@
 		(in_pos_files yes)
 		(dnp no)
-		(property "Reference" "R37"
-			(at 185.674 230.124 0)
+		(property "Reference" "R47"
+			(at 192.786 225.044 0)
 			(show_name no)
 			(do_not_autoplace no)
@@
 		)
 		(property "Value" "100Ω"
-			(at 184.404 231.902 0)
+			(at 191.008 223.774 0)
 			(show_name no)
 			(do_not_autoplace no)
@@
 		)
 		(property "Footprint" "Resistor_SMD:R_0402_1005Metric"
-			(at 190.754 231.394 90)
+			(at 191.516 230.124 90)
 			(hide yes)
 			(show_name no)
@@
 			(project "PelletPirate_V5"
 				(path "/0182ac56-03c6-4c14-8ead-12e31828f094"
-					(reference "R37")
+					(reference "R47")
 					(unit 1)
 				)
@@
 		(in_pos_files yes)
 		(dnp no)
-		(property "Reference" "R36"
+		(property "Reference" "R44"
 			(at 192.532 161.798 90)
 			(show_name no)
@@
 			(project "PelletPirate_V5"
 				(path "/0182ac56-03c6-4c14-8ead-12e31828f094"
-					(reference "R36")
+					(reference "R44")
 					(unit 1)
 				)
@@
 		(in_pos_files yes)
 		(dnp no)
-		(property "Reference" "R38"
+		(property "Reference" "R35"
 			(at 242.57 213.868 0)
 			(show_name no)
@@
 			(project "PelletPirate_V5"
 				(path "/0182ac56-03c6-4c14-8ead-12e31828f094"
-					(reference "R38")
+					(reference "R35")
 					(unit 1)
 				)
@@
 		(in_pos_files yes)
 		(dnp no)
-		(property "Reference" "R32"
+		(property "Reference" "R45"
 			(at 150.876 176.53 90)
 			(show_name no)
@@
 			(project "PelletPirate_V5"
 				(path "/0182ac56-03c6-4c14-8ead-12e31828f094"
-					(reference "R32")
+					(reference "R45")
 					(unit 1)
 				)
@@
 			)
 		)
-		(property "Footprint" "PBO-5F-12_PP_Try2:PBO-5F-12_pp2"
+		(property "Footprint" "NewPBO-5F-12-try:CONV_PBO-5F-12_AUDIT_FLYMAN"
 			(at 184.15 39.37 0)
 			(hide yes)
@@
 		(in_pos_files yes)
 		(dnp no)
-		(property "Reference" "WirePad6"
+		(property "Reference" "WirePad5"
 			(at 97.028 282.448 0)
 			(hide yes)
@@
 			(project "PelletPirate_V5"
 				(path "/0182ac56-03c6-4c14-8ead-12e31828f094"
-					(reference "WirePad6")
+					(reference "WirePad5")
 					(unit 1)
 				)
@@
 		(in_pos_files yes)
 		(dnp no)
-		(property "Reference" "R34"
+		(property "Reference" "R33"
 			(at 172.466 201.676 0)
 			(show_name no)
@@
 			(project "PelletPirate_V5"
 				(path "/0182ac56-03c6-4c14-8ead-12e31828f094"
-					(reference "R34")
+					(reference "R33")
 					(unit 1)
 				)
@@
 		(in_pos_files yes)
 		(dnp no)
-		(property "Reference" "R44"
+		(property "Reference" "R42"
 			(at 42.164 295.656 90)
 			(show_name no)
@@
 			(project "PelletPirate_V5"
 				(path "/0182ac56-03c6-4c14-8ead-12e31828f094"
-					(reference "R44")
+					(reference "R42")
 					(unit 1)
 				)
@@
 			)
 		)
-		(property "Footprint" "Connector_Wire:SolderWire-2.5sqmm_1x01_D2.4mm_OD3.6mm"
+		(property "Footprint" "Connector_Wire:SolderWire-1.5sqmm_1x01_D1.7mm_OD3mm"
 			(at 105.41 218.44 0)
 			(hide yes)
@@
 			)
 		)
-		(property "Footprint" "Connector_Wire:SolderWire-2.5sqmm_1x01_D2.4mm_OD4.4mm"
+		(property "Footprint" "Connector_Wire:SolderWire-1.5sqmm_1x01_D1.7mm_OD3mm"
 			(at 63.5 34.29 0)
 			(hide yes)
