File: KiCad/pelletpirate_V5/PelletPirate_V5.kicad_sch (KiCad schematic)
At the start: 128 parts, among them J1 SJ1-3523NG_Jack_PP, J10 TB002-500-02BE, J2 SJ1-3523NG_Jack_PP, J3 SJ1-3523NG_Jack_PP, J4 SJ1-3523NG_Jack_PP, J5 SJ1-3523NG_Jack_PP, J6 Conn_01x04, J7 Conn_01x04_Socket, J9 USB4145-03-0070-C_REVA2, T1 BTA12-Triac, T2 BTA12-Triac, T3 BTA12-600BWRG, U1 USBLC6-2SC6, U3 H11AA1M

Commit message: V5 DRC Clean / ERC Clean
USB-C corner closed out:
- USB4145 footprint copper verified against GCT drawing (unproven-source flag retired)
- Per-pad solder mask expansion zeroed -> real 0.2mm mask dams (10 aperture-bridge DRC cleared)
- Hidden power-in duplicate pins (A9/A12/B9/B12) converted to hidden passive (shield-pin style); implicit VBUS_A/GND_A global net injection eliminated
- Net renamed VBUS_A -> /VBUS; USB netclass pattern fixed to /VBUS (silent class dropout repaired)
- ERC 0/0 verified via kicad-cli at all severities; DRC clean with fresh zone fills
- Top-half placement plan sketch added (MAX tiles under jacks, ESP south, U3 east, PS3 to FPC backlight end)

Co-Authored-By: Claude Fable 5 <noreply@anthropic.com>
Parts:
- C21, C22, C23, C24, C25, C26, C27, C28, C29, C30, C31, C32, C33, C34, C35: footprint Capacitor_SMD:C_0805_2012Metric -> Capacitor_SMD:C_0402_1005Metric; LINK (none) -> https://www.digikey.com/en/products/detail/samsung-electro-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; MF (none) -> YAGEO; MP (none) -> CL05B104KO5NNNC
- D2: footprint STPS0540Z_Schotty Diode LED:SOD-123 -> STPS0540Z_Schotty Diode LED:D2-Footprint-Flyman
- R9: footprint Resistor_SMD:R_0805_2012Metric -> Resistor_SMD:R_0805_2012Metric_Pad1.20x1.40mm_HandSolder
- WirePad2: value NEUTRAL-In -> (N)-in
- renumbered J9 to J8, J10 to J9
Connections:
- net +12V: now also C11.1; no longer C11.2
- net GND: now also C11.2; no longer C11.1
- net MAX1_CS: now also ESP1.4 (IO4); no longer ESP1.23 (IO21)
- net MAX5_CS: now also ESP1.23 (IO21); no longer ESP1.4 (IO4)
- net VBUS_A renamed VBUS

Commit message: V5 pre-library-localization safety checkpoint
- Audit remediation complete: corridor items 1-5 + 7 closed (LED/SPI reroute,
  J4 overlays, CS nudges, MAX5_CS old run deleted, ZC_DET+GND test points TP1/TP2,
  parity field sync). ERC 0/0, DRC 0/0, parity 0.
- New-connector audit: J8 USB4145 + J9 TB002 verified against datasheets;
  finding F1 open (stake variant 0070 -> 0170 swap pending)
- USB_try2: staged 0170 symbol (hidden-pin-fixed) + footprint + STEP
- V5_Library_Localization_Plan.md: proposed plan, not yet executed

Co-Authored-By: Claude Fable 5 <noreply@anthropic.com>
Parts:
- added TP1, TP2: TestPoint, TestPoint:TestPoint_THTPad_D1.5mm_Drill0.7mm, symbol Connector:TestPoint
- C10, C8: LINK (none) -> https://www.digikey.com/en/products/detail/kemet/C1206C106K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
- C11, C14: LINK (none) -> https://www.digikey.com/en/products/detail/kemet/C0805C104K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; MF (none) -> KEMET; MP (none) -> C0805C104K5RACTU
- C12: LINK (none) -> https://www.digikey.com/en/products/detail/vishay-beyschlag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; MF (none) -> VISHAY; MP (none) -> VY2102M29Y5US63V7
- C13: LINK (none) -> https://www.digikey.com/en/products/detail/kemet/A750MS477M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; MF (none) -> KEMET; MP (none) -> A750MS477M1EAAE015
- C15: LINK (none) -> https://www.digikey.com/en/products/detail/kyocera-avx/RPF0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; MF (none) -> KYOCERA AVX; MP (none) -> RPF0811221M035K
- C16: LINK (none) -> https://www.digikey.com/en/products/detail/kemet/C0805C105K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; MF (none) -> KEMET; MP (none) -> C0805C105K5RACTU
- C18, C19, C20: LINK (none) -> https://www.digikey.com/en/products/detail/murata-electroni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; MF (none) -> MURATA; MP (none) -> GRM31CZ71C226ME15L
- C21, C22, C23, C24, C25, C26, C27, C28, C29, C30, C31, C32, C33, C34, C35: MF YAGEO -> Samsung
- C36: LINK (none) -> https://www.digikey.com/en/products/detail/kemet/C0805C224K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; MF (none) -> KEMET; MP (none) -> C0805C224K5RACTU
- C38: LINK https://www.digikey.com/en/products/detail/kemet/C1206C106K3RACTU/3317648 -> https://www.digikey.com/en/products/detail/kemet/C1206C106K3RACTU/3317648
- C4: LINK (none) -> https://www.digikey.com/en/products/detail/kemet/R46KF31000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; MF (none) -> KEMET; MP (none) -> R46KF310000M1M
- C5, C6, C7: LINK (none) -> https://www.digikey.com/en/products/detail/vishay-beyschlag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
- D1: LINK (none) -> https://www.digikey.com/en/products/detail/littelfuse-inc/S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
- D2: LINK (none) -> https://www.digikey.com/en/products/detail/stmicroelectroni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
- FPC1: LINK (none) -> https://www.digikey.com/en/products/detail/hirose-electric-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
- J8: value USB4145-03-0070-C_REVA2 -> USB4145-03-0170-C; Check_prices https://www.snapeda.com/parts/USB4145-03-0070-C/Global+Conn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 -> (none); LINK (none) -> https://www.digikey.com/en/products/detail/gct/USB4145-03-0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; MP USB4145-03-0070-C -> USB4145-03-0170-C; SNAPEDA_PN USB4145-03-0070-C -> USB4145-03-0170-C; SnapEDA_Link https://www.snapeda.com/parts/USB4145-03-0070-C/Global+Conn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 -> https://www.digikey.com/en/products/detail/gct/USB4145-03-0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
- L1, L2: LINK (none) -> https://www.digikey.com/en/products/detail/murata-electroni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
- L3: LINK (none) -> https://www.digikey.com/en/products/detail/bourns-inc/SRR40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
- LF1: LINK (none) -> https://www.digikey.com/en/products/detail/kemet/SSRH7H-M05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; MF (none) -> KEMET; MP (none) -> SSRH7H-M05408
- MAX1, MAX2, MAX3, MAX4, MAX5: LINK (none) -> https://www.digikey.com/en/products/detail/analog-devices-i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; MF (none) -> ANALOG DEVICES; MP (none) -> MAX31865ATP+
- MOC1, MOC2: LINK (none) -> https://www.digikey.com/en/products/detail/onsemi/MOC3063M/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; MF (none) -> ONSEMI; MP (none) -> MOC3063M
- MOV1: LINK (none) -> https://www.digikey.com/en/products/detail/bourns-inc/MOV-1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; MF (none) -> BOURNS; MP (none) -> MOV-14D561K
- PS1: LINK (none) -> https://www.digikey.com/en/products/detail/bel-power-soluti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
- PS2, PS3: LINK (none) -> https://www.digikey.com/en/products/detail/texas-instrument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
- R17: LINK (none) -> https://www.digikey.com/en/products/detail/yageo/RC1206FR-0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; MF (none) -> YAGEO; MP (none) -> RC1206FR-074R99L
- R21, R22, R23, R24, R25: LINK (none) -> https://www.digikey.com/en/products/detail/yageo/RT1206BRD0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; MF (none) -> YAGEO; MP (none) -> RT1206BRD07400RL
- R7, R8: LINK (none) -> https://www.digikey.com/en/products/detail/panasonic-indust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
- T1, T2: value BTA12-Triac -> BTA12-600BWRG; LINK (none) -> https://www.digikey.com/en/products/detail/stmicroelectroni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; MF (none) -> STMicroelectronics; MP (none) -> BTA12-600BWRG
- T3: LINK https://www.digikey.com/en/products/detail/stmicroelectronics/BTA12-600BWRG/654429 -> https://www.digikey.com/en/products/detail/stmicroelectronics/BTA12-600BWRG/654429; MP BTA12-600BWRG -> BTA12-600BWRG
Connections:
- net GND: now also TP2.1
- net ZC_DET: now also TP1.1

Commit message: V5 pre-BOM-fill checkpoint: J8 0170 swap in sch+board, footprint/mask cleanups, BOM fill table
Co-Authored-By: Claude Fable 5 <noreply@anthropic.com>
Parts:
- J8: footprint USB_try2:GCT_USB4145-03-0070-C_REVA2 -> USB_try2:GCT_USB4145-03-0170-C
Changed lines of the file:
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@@
 			)
 		)
-		(property "Footprint" "USB_try2:GCT_USB4145-03-0070-C_REVA2"
+		(property "Footprint" "USB_try2:GCT_USB4145-03-0170-C"
 			(at 334.01 200.66 0)
 			(hide yes)

Commit message: V5 BOM complete: all fields filled, zero gaps
Scripted field fill (approved by user, KiCad closed, verified via kicad-cli):
- 28 parts filled with MF/MP/LINK (V4-sourced parts value+footprint matched;
  new parts DigiKey-verified: B32921C3103M000 X2 snubber caps, ERJ-1TYJ390U,
  RC0805FR-07330RL, RC0805FR-07100KL)
- LINK fills for J1-J5/J9/F1; J4 cache-collision handled (insert into instance)
- R6 omega normalized to match R9 (BOM line un-split)
- TP1/TP2 excluded from BOM
Final: 117 BOM rows, 0 missing MP/MF/LINK, ERC 0

Co-Authored-By: Claude Fable 5 <noreply@anthropic.com>
Parts:
- C1, C2, C3: LINK (none) -> https://www.digikey.com/en/products/detail/epcos-tdk-electr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; MF (none) -> EPCOS - TDK; MP (none) -> B32921C3103M000
- C10, C8: LINK https://www.digikey.com/en/products/detail/kemet/C1206C106K3RACTU/3317648 -> https://www.digikey.com/en/products/detail/kemet/C1206C106K3RACTU/3317648; MF (none) -> KEMET; MP (none) -> C1206C106K3RACTU
- C5, C6: MF (none) -> VISHAY; MP (none) -> VY2471K29Y5SS63V7
- C7: LINK https://www.digikey.com/en/products/detail/vishay-beyschlag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 -> https://www.digikey.com/en/products/detail/rubycon/450BXG15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; MF (none) -> Rubycon; MP (none) -> 450BXG15MEFC10X20
- C9: LINK (none) -> https://www.digikey.com/en/products/detail/kemet/C0402C104K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; MF (none) -> KEMET; MP (none) -> C0402C104K3RACTU
- F1: LINK (none) -> https://www.digikey.com/en/products/result?keywords=0031.82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
- J1, J2, J3, J4, J5, J9: LINK (none) -> https://www.digikey.com/en/products/detail/same-sky-formerl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
- J6: LINK (none) -> https://www.digikey.com/en/products/detail/hirose-electric-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; MF (none) -> Hirose Electric Co Ltd; MP (none) -> DF13-4P-1.25DSA(25)
- R1, R2, R3: LINK (none) -> https://www.digikey.com/en/products/detail/panasonic-electr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; MF (none) -> PANASONIC; MP (none) -> ERJ-1TYJ390U
- R15: LINK (none) -> https://www.digikey.com/en/products/detail/yageo/RC0805FR-0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; MF (none) -> YAGEO; MP (none) -> RC0805FR-07100KL
- R16: LINK (none) -> https://www.digikey.com/en/products/detail/yageo/RC0603FR-0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; MF (none) -> YAGEO; MP (none) -> RC0603FR-07100KL
- R19: LINK (none) -> https://www.digikey.com/en/products/detail/yageo/RC0805FR-0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; MF (none) -> YAGEO; MP (none) -> RC0805FR-0733K2L
- R20: LINK (none) -> https://www.digikey.com/en/products/detail/yageo/RC0402FR-0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; MF (none) -> YAGEO; MP (none) -> RC0402FR-0710KL
- R26, R27, R4, R5: LINK (none) -> https://www.digikey.com/en/products/detail/vishay-dale/CRCW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; MF (none) -> VISHAY; MP (none) -> CRCW1206360RFKEA
- R6: value 180Ω -> 180Ω
- R7, R8: LINK https://www.digikey.com/en/products/detail/panasonic-indust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 -> https://www.digikey.com/en/products/detail/yageo/RC0805FR-0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; MF (none) -> YAGEO; MP (none) -> RC0805FR-07330RL
- TP1, TP2: now left out of the parts list
