File: KiCad/pelletpirate_V5v1/PelletPirate_V5v1.kicad_sch (KiCad schematic)
At the start: 130 parts, among them J1 SJ1-3523NG_Jack_PP, J2 SJ1-3523NG_Jack_PP, J3 SJ1-3523NG_Jack_PP, J4 SJ1-3523NG_Jack_PP, J5 SJ1-3523NG_Jack_PP, J6 Conn_01x04, J7 Conn_01x04_Socket, J8 USB4145-03-0170-C, J9 TB002-500-02BE, T1 BTA12-600BWRG, T2 BTA12-600BWRG, T3 BTA12-600BWRG, U1 USBLC6-2SC6, U3 H11AA1M

Commit message: V5v1: PS1 MF harmonized to CUI Inc. (Bel/CUI dual-brand, same product - not an error fix)
Co-Authored-By: Claude Fable 5 <noreply@anthropic.com>
Parts:
- PS1: MF Bel Fuse -> CUI Inc.
Changed lines of the file:
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@@
 			)
 		)
-		(property "MF" "Bel Fuse"
+		(property "MF" "CUI Inc."
 			(at 184.15 39.37 0)
 			(hide yes)

Commit message: Fix C9/R20 package mismatches: 0402 MPNs on 0805 footprints -> 0805 parts
- PCBWay BOM: C9 -> C0805C104K3RACTU, R20 -> RC0805FR-0710KL (both DK-verified in stock)
- V5v1 sch fields updated to match copper; backlog notes the 0402 shrink path for V5.1
- Root cause: V4 value-matching missed footprint check on these 2 of 61 lines

Co-Authored-By: Claude Fable 5 <noreply@anthropic.com>
Parts:
- C9: LINK https://www.digikey.com/en/products/detail/kemet/C0402C104K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 -> https://www.digikey.com/en/products/detail/kemet/C0805C104K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; MP C0402C104K3RACTU -> C0805C104K3RACTU
- R20: LINK https://www.digikey.com/en/products/detail/yageo/RC0402FR-0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 -> https://www.digikey.com/en/products/detail/yageo/RC0805FR-0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; MP RC0402FR-0710KL -> RC0805FR-0710KL
Changed lines of the file:
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@@
 			)
 		)
-		(property "MP" "RC0402FR-0710KL"
+		(property "MP" "RC0805FR-0710KL"
 			(at 123.19 101.6 0)
 			(effects
@@
 			)
 		)
-		(property "LINK" "https://www.digikey.com/en/products/detail/yageo/RC0402FR-0710KL/726523"
+		(property "LINK" "https://www.digikey.com/en/products/detail/yageo/RC0805FR-0710KL/727535"
 			(at 123.19 101.6 0)
 			(effects
@@
 			)
 		)
-		(property "MP" "C0402C104K3RACTU"
+		(property "MP" "C0805C104K3RACTU"
 			(at 186.69 92.71 0)
 			(effects
@@
 			)
 		)
-		(property "LINK" "https://www.digikey.com/en/products/detail/kemet/C0402C104K3RACTU/6697176"
+		(property "LINK" "https://www.digikey.com/en/products/detail/kemet/C0805C104K3RACTU/411167"
 			(at 186.69 92.71 0)
 			(effects

Commit message: V5v1 re-cloned fresh from as-ordered V5 (supersedes stale 80a9e8e clone)
V5 = frozen as-sent-to-PCBWay reference; V5v1 = working copy for all future tweaks.
Core files renamed + all internal refs patched (142 pcb sheetfile, 203 sch project,
pro meta/sheets/bom-path now local). Excluded: backups, archive_to_delete, PCBWay pkg.
ENHANCEMENT_BACKLOG carried over. Verified from new dir: ERC 0, DRC 0, unconnected 0.

Co-Authored-By: Claude Fable 5 <noreply@anthropic.com>
Parts:
- added C43: 0.1µF 25V, Capacitor_SMD:C_0402_1005Metric, symbol Device:C
- added C44, C45, C47: 22µF 16V, Capacitor_SMD:C_1206_3216Metric, symbol Device:C
- added C46: 0.1µF 16V, Capacitor_SMD:C_0402_1005Metric, symbol Device:C
- added C48: 220µF 35V, Capacitor_THT:CP_Radial_D8.0mm_P3.50mm, symbol Device:C_Small_US
- added FL1: BLM21PG221SN1D, Ferrite_Bead:BEADC2012X105N, symbol BLM21PG221SN1D:BLM21PG221SN1D
- added L5: BLM31PG601SN1L, Ferrite_Bead_12V_Flyman:BEADC3216X130N_flyman, symbol BLM31PG601SN1L_flyman:BLM31PG601SN1L
- added R48, R49, R50, R51: 33Ω, Resistor_SMD:R_0402_1005Metric, symbol Device:R_US
- C38: LINK https://www.digikey.com/en/products/detail/kemet/C1206C106K3RACTU/3317648 -> https://www.digikey.com/en/products/detail/kemet/C1206C106K3RACTU/3317648; MP C1206C106K3RACTU -> C1206C106K3RACTU
- C39: value 0.1µF 25V -> 1.0µF 25V; footprint Capacitor_SMD:C_0402_1005Metric -> Capacitor_SMD:C_0603_1608Metric; LINK https://www.digikey.com/en/products/detail/kemet/C0402C104K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 -> https://www.digikey.com/en/products/detail/kemet/C0603C105K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; MP C0402C104K3RACTU -> C0603C105K3RACTU
- C9: footprint Capacitor_SMD:C_0805_2012Metric -> Capacitor_SMD:C_0402_1005Metric; LINK https://www.digikey.com/en/products/detail/kemet/C0805C104K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 -> https://www.digikey.com/en/products/detail/kemet/C0402C104K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; MP C0805C104K3RACTU -> C0402C104K3RACTU
- PS1: MF CUI Inc. -> Bel Fuse
- R20: footprint Resistor_SMD:R_0805_2012Metric_Pad1.20x1.40mm_HandSolder -> Resistor_SMD:R_0805_2012Metric
Connections:
- net +12V: now also C48.1, L5.2; no longer C15.1, D1.1, L1.2
- net +3.3V: now also C44.1, C45.1, FL1.1; no longer C40.2, FPC1.3, FPC1.34, FPC1.35
- net ALL_SCLK: now also R49.2; no longer ESP1.33 (IO40)
- net ALL_SDI: now also R48.2; no longer ESP1.32 (IO39)
- net GND: now also C40.2, C43.2, C44.2, C45.2, C46.1, C47.2, C48.2
- net LCD_CS: now also R50.2; no longer ESP1.9 (IO16)
- net LCD_DC: now also R51.2; no longer ESP1.11 (IO18)
- net VBUS: now also C43.1
- new net: C15.1, D1.1, L1.2, L5.1
- new net: ESP1.11 (IO18), R51.1
- new net: ESP1.32 (IO39), R48.1
- new net: ESP1.33 (IO40), R49.1
- new net: ESP1.9 (IO16), R50.1
- new net 3V3_LCD: C46.2, C47.1, FL1.2, FPC1.3, FPC1.34, FPC1.35
Other:
- moved on the sheet: C15, C17, C37, C38, C40, C42, J7, R41, R42, R43, TP1, TP2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
